Commit message: Created control pakage

File: hexapod_description_pkg/urdf/hexapod_gazebo_transmission.xacro (robot description, xacro)
@@ -1,10 +1,17 @@
 <?xml version="1.0"?>
 <robot xmlns:xacro="http://ros.org/wiki/xacro" name="hexapod">
-<xacro:macro name="default_inertial" params="mass">
+<!-- ros_control plugin -->
+<gazebo>
+  <plugin name="gazebo_ros_control" filename="libgazebo_ros_control.so">
+    <robotNamespace>/hexapod</robotNamespace>
+  </plugin>
+</gazebo>
+    <xacro:macro name="default_inertial" params="mass">
                <inertial>
-                       <mass value="${mass}" />
-                       <inertia ixx="1.0" ixy="0.0" ixz="0.0"
-                                iyy="1.0" iyz="0.0"
-                                izz="1.0" />
+                        <origin xyz="0 0 1" rpy="0 0 0"/>
+                        <mass value="${mass}" />
+                        <inertia ixx="0.5" ixy="0.0" ixz="0.0"
+                                 iyy="0.5" iyz="0.0"
+                                 izz="0.5" />
                </inertial>
     </xacro:macro>
@@ -115,4 +122,5 @@
             <turnGravityOff>false</turnGravityOff>
         </link>
+        <!-- Joints description -->
          <joint name="leg_center_joint_${side}${num}" type="fixed">
             <origin xyz="${x} ${y} 0" rpy="0 0 0" />
@@ -146,4 +154,35 @@
             <child  link="tibia_foot_${side}${num}" />
         </joint>
+        <!-- Transmissions for all joints -->
+        <transmission name="coxa_trans_${side}${num}">
+            <type>transmission_interface/SimpleTransmission</type>
+            <joint name="coxa_joint_${side}${num}">
+                <hardwareInterface>EffortJointInterface</hardwareInterface>
+            </joint>
+            <actuator name="motor_coxa_${side}${num}">
+                <hardwareInterface>EffortJointInterface</hardwareInterface>
+                <mechanicalReduction>1</mechanicalReduction>
+            </actuator>
+        </transmission>
+        <transmission name="femur_trans_${side}${num}">
+            <type>transmission_interface/SimpleTransmission</type>
+            <joint name="femur_joint_${side}${num}">
+                <hardwareInterface>EffortJointInterface</hardwareInterface>
+            </joint>
+            <actuator name="motor_femur_${side}${num}">
+                <hardwareInterface>EffortJointInterface</hardwareInterface>
+                <mechanicalReduction>1</mechanicalReduction>
+            </actuator>
+        </transmission>
+        <transmission name="tibia_trans_${side}${num}">
+            <type>transmission_interface/SimpleTransmission</type>
+            <joint name="tibia_joint_${side}${num}">
+                <hardwareInterface>EffortJointInterface</hardwareInterface>
+            </joint>
+            <actuator name="motor_tibia_${side}${num}">
+                <hardwareInterface>EffortJointInterface</hardwareInterface>
+                <mechanicalReduction>1</mechanicalReduction>
+            </actuator>
+        </transmission>
     </xacro:macro>
     <!-- Build robot using leg maros and thorax -->

Commit message: Added base for forwards moving script

File: hexapod_description_pkg/urdf/hexapod_gazebo_transmission.xacro (robot description, xacro)
@@ -47,6 +47,6 @@
     <xacro:property name="joint_lower_limit" value="-${1.5}" />
     <xacro:property name="joint_upper_limit" value="${1.5}"  />
-    <xacro:property name="joint_effort"      value="10000"   />
-    <xacro:property name="joint_velocity"    value="100"     />
+    <xacro:property name="joint_effort"      value="90"   />
+    <xacro:property name="joint_velocity"    value="900"     />
     <!-- Leg Builer Macro -->
     <xacro:macro name="leg" params="side num x y angle">

Commit message: Identified problem in unbalaced step

File: hexapod_description_pkg/urdf/hexapod_gazebo_transmission.xacro (robot description, xacro)
@@ -133,5 +133,6 @@
             <child  link="coxa_${side}${num}" />
             <axis xyz="0 0 -1" />
-            <limit lower="${joint_lower_limit}" upper="${joint_upper_limit}" effort="${joint_effort}" velocity="${joint_velocity}" />
+            <limit lower="${joint_lower_limit}" upper="${joint_upper_limit}"
+                   effort="${joint_effort}" velocity="${joint_velocity}" />
         </joint>
         <joint name="femur_joint_${side}${num}" type="revolute">
@@ -140,5 +141,6 @@
             <child  link="femur_${side}${num}" />
             <axis   xyz="0 0 -1" />
-            <limit lower="${joint_lower_limit}" upper="${joint_upper_limit}" effort="${joint_effort}" velocity="${joint_velocity}" />
+            <limit lower="${joint_lower_limit}" upper="${joint_upper_limit}"
+                   effort="${joint_effort}" velocity="${joint_velocity}" />
         </joint>
         <joint name="tibia_joint_${side}${num}" type="revolute">
@@ -147,5 +149,6 @@
             <child  link="tibia_${side}${num}" />
             <axis   xyz="0 0 1" />
-            <limit  lower="${joint_lower_limit}" upper="${joint_upper_limit}" effort="${joint_effort}" velocity="${joint_velocity}" />
+            <limit  lower="${joint_lower_limit}" upper="${joint_upper_limit}"
+                    effort="${joint_effort}" velocity="${joint_velocity}" />
         </joint>
         <joint name="tibia_foot_joint_${side}${num}" type="fixed">

Commit message: keeping straight line

File: hexapod_description_pkg/urdf/hexapod_gazebo_transmission.xacro (robot description, xacro)
@@ -11,7 +11,7 @@
                         <origin xyz="0 0 1" rpy="0 0 0"/>
                         <mass value="${mass}" />
-                        <inertia ixx="0.5" ixy="0.0" ixz="0.0"
-                                 iyy="0.5" iyz="0.0"
-                                 izz="0.5" />
+                        <inertia ixx="0.1" ixy="0.0" ixz="0.0"
+                                 iyy="0.1" iyz="0.0"
+                                 izz="0.1" />
                </inertial>
     </xacro:macro>
@@ -39,5 +39,5 @@
             </geometry>
         </collision>
-        <xacro:default_inertial mass="10"/>
+        <xacro:default_inertial mass="1"/>
         <turnGravityOff>false</turnGravityOff>
     </link>
